Commit message: chiaa

File: src/robotino_webots/urdf/Robotino3.urdf (robot description, URDF)
Before this commit: robot /home/oscar/Robotino3.urdf, 28 links, 27 joints
Links:
- link wheel0_link: geometry collision mesh filename=package://webots/projects/robots/festo/robotino3/protos/mes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; visual mesh filename=package://webots/projects/robets/festo/robotino3/protos/mes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
- link wheel1_link: geometry collision mesh filename=package://webots/projects/robots/festo/robotino3/protos/mes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; visual mesh filename=package://webots/projects/robots/festo/robotino3/protos/mes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
- link wheel2_link: geometry collision mesh filename=package://webots/projects/robots/festo/robotino3/protos/mes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; visual mesh filename=package://webots/projects/robots/festo/robotino3/protos/mes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

Commit message: amcl died, floor good

File: src/robotino_webots/urdf/Robotino3.urdf (robot description, URDF)
Before this commit: robot /home/oscar/Robotino3.urdf, 28 links, 27 joints
Links:
- link base_link: geometry collision cylinder length=0.276 radius=0.2266; visual cylinder length=0.276 radius=0.2266
- link wheel0_link: geometry collision cylinder length=0.01 radius=0.063; visual cylinder length=0.01 radius=0.063
- link wheel1_link: geometry collision cylinder length=0.01 radius=0.063; visual cylinder length=0.01 radius=0.063
- link wheel2_link: geometry collision cylinder length=0.01 radius=0.063; visual cylinder length=0.01 radius=0.063

Commit message: amcl works

File: src/robotino_webots/urdf/Robotino3.urdf (robot description, URDF)
Before this commit: robot /home/oscar/Robotino3.urdf, 28 links, 27 joints
Links:
- link base_link: geometry collision cylinder length=0.276 radius=0.2266; visual mesh filename=package://rto_description/meshes/parts/robotino_base.dae scale=0.01 0.01 0.01
- link wheel0_link: geometry collision cylinder length=0.01 radius=0.063; visual mesh filename=package://rto_description/meshes/parts/robotino_wheel.dae scale=0.01 0.01 0.01
- link wheel1_link: geometry collision cylinder length=0.01 radius=0.063; visual mesh filename=package://rto_description/meshes/parts/robotino_wheel.dae scale=0.01 0.01 0.01
- link wheel2_link: geometry collision cylinder length=0.01 radius=0.063; visual mesh filename=package://rto_description/meshes/parts/robotino_wheel.dae scale=0.01 0.01 0.01
